File: L298 Motor Driver.sch (EAGLE design)
At the start: 15 parts, among them IC1 L298, J1 1X2-3.5MM, J2 1X2-3.5MM, J3 1X2-3.5MM

Commit message: Added info to title block
Other:
- note added: "1"
- note added: "L298 Dual H-Bridge Motor Driver"
Changed lines of the file:
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@@
 <sheet>
 <plain>
+<text x="175.26" y="30.48" size="2.54" layer="94">L298 Dual H-Bridge Motor Driver</text>
+<text x="266.7" y="7.62" size="2.54" layer="94">1</text>
 </plain>
 <instances>

Commit message: Added info to title block
Other:
- note added: "without current sense resistors"
- note removed: "1"
Changed lines of the file:
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@@
 <plain>
 <text x="175.26" y="30.48" size="2.54" layer="94">L298 Dual H-Bridge Motor Driver</text>
-<text x="266.7" y="7.62" size="2.54" layer="94">1</text>
+<text x="175.26" y="25.4" size="2.54" layer="94">without current sense resistors</text>
 </plain>
 <instances>
